Commit message: Revert "Changed joint names to original bd names for compatibility"
This reverts commit 98ae067835cb0afbe43e1e540a719851c9854c6c.

File: hector_spot_description/urdf/spot_base.urdf.xacro (robot description, xacro)
@@ -52,5 +52,5 @@
         </inertial>
     </link>
-    <joint name="fl.hx" type="revolute">
+    <joint name="front_left_hip_x" type="revolute">
         <origin xyz="0.29785 0.05500 0.00000" rpy="0 0 0" />
         <axis xyz="1 0 0" />
@@ -75,5 +75,5 @@
         </inertial>
     </link>
-    <joint name="fl.hy" type="revolute">
+    <joint name="front_left_hip_y" type="revolute">
         <origin xyz="0.0 0.110945 0.0" rpy="0 0 0" />
         <axis xyz="0 1 0" />
@@ -98,5 +98,5 @@
         </inertial>
     </link>
-    <joint name="fl.kn" type="revolute">
+    <joint name="front_left_knee" type="revolute">
         <origin xyz="0.025 0.000 -0.3205" rpy="0 0 0" />
         <axis xyz="0 1 0" />
@@ -121,5 +121,5 @@
         </inertial>
     </link>
-    <joint name="fr.hx" type="revolute">
+    <joint name="front_right_hip_x" type="revolute">
         <origin xyz="0.29785 -0.05500 0.00000" rpy="0 0 0" />
         <axis xyz="1 0 0" />
@@ -144,5 +144,5 @@
         </inertial>
     </link>
-    <joint name="fr.hy" type="revolute">
+    <joint name="front_right_hip_y" type="revolute">
         <origin xyz="0.0 -0.110945 0.0" rpy="0 0 0" />
         <axis xyz="0 1 0" />
@@ -167,5 +167,5 @@
         </inertial>
     </link>
-    <joint name="fr.kn" type="revolute">
+    <joint name="front_right_knee" type="revolute">
         <origin xyz="0.025 0.000 -0.3205" rpy="0 0 0" />
         <axis xyz="0 1 0" />
@@ -190,5 +190,5 @@
         </inertial>
     </link>
-    <joint name="hl.hx" type="revolute">
+    <joint name="rear_left_hip_x" type="revolute">
         <origin xyz="-0.29785 0.05500 0.00000" rpy="0 0 0" />
         <axis xyz="1 0 0" />
@@ -213,5 +213,5 @@
         </inertial>
     </link>
-    <joint name="hl.hy" type="revolute">
+    <joint name="rear_left_hip_y" type="revolute">
         <origin xyz="0.0 0.110945 0.0" rpy="0 0 0" />
         <axis xyz="0 1 0" />
@@ -236,5 +236,5 @@
         </inertial>
     </link>
-    <joint name="hl.kn" type="revolute">
+    <joint name="rear_left_knee" type="revolute">
         <origin xyz="0.025 0.000 -0.3205" rpy="0 0 0" />
         <axis xyz="0 1 0" />
@@ -259,5 +259,5 @@
         </inertial>
     </link>
-    <joint name="hr.hx" type="revolute">
+    <joint name="rear_right_hip_x" type="revolute">
         <origin xyz="-0.29785 -0.05500 0.00000" rpy="0 0 0" />
         <axis xyz="1 0 0" />
@@ -282,5 +282,5 @@
         </inertial>
     </link>
-    <joint name="hr.hy" type="revolute">
+    <joint name="rear_right_hip_y" type="revolute">
         <origin xyz="0.0 -0.110945 0.0" rpy="0 0 0" />
         <axis xyz="0 1 0" />
@@ -305,5 +305,5 @@
         </inertial>
     </link>
-    <joint name="hr.kn" type="revolute">
+    <joint name="rear_right_knee" type="revolute">
         <origin xyz="0.025 0.000 -0.3205" rpy="0 0 0" />
         <axis xyz="0 1 0" />

Commit message: Reversed body -> base_link transform to be a chain

File: hector_spot_description/urdf/spot_base.urdf.xacro (robot description, xacro)
@@ -2,4 +2,9 @@
 <robot name="spot_base" xmlns:xacro="http://ros.org/wiki/xacro">
   <xacro:macro name="spot_base">
+    <link name="base_link"/>
+    <joint name="base_link_joint" type="fixed">
+        <parent link="base_link" />
+        <child link="body" />
+    </joint>
     <link name="body">
         <visual>
@@ -18,10 +23,4 @@
         </inertial>
     </link>
-    <link name="base_link"/>
-    <joint name="base_link_joint" type="fixed">
-        <origin xyz="0 0 0" rpy="0 0 0" />
-        <parent link="body" />
-        <child link="base_link" />
-    </joint>
     <link name="front_rail"/>
     <joint name="front_rail_joint" type="fixed">

Commit message: Refactored legs into macro
from https://github.com/chvmp/spot_ros/tree/gazebo

File: hector_spot_description/urdf/spot_base.urdf.xacro (robot description, xacro)
@@ -1,4 +1,27 @@
 <?xml version="1.0"?>
 <robot name="spot_base" xmlns:xacro="http://ros.org/wiki/xacro">
+  <xacro:include filename="$(find hector_spot_description)/urdf/spot_leg.urdf.xacro" />
+  <xacro:property name="base_to_hip_x" value="0.29785" />
+  <xacro:property name="base_to_hip_y" value="0.05500" />
+  <xacro:property name="hip_to_upper_leg_y" value="0.110945" />
+  <xacro:property name="upper_leg_to_lower_leg_x" value="0.025" />
+  <xacro:property name="upper_leg_to_lower_leg_z" value="0.3205" />
+  <xacro:property name="lower_leg_to_foot_z" value="0.37" />
+  <xacro:property name="base_mass" value="16.0" />
+  <xacro:property name="base_length" value="0.86" />
+  <xacro:property name="base_width" value="0.21" />
+  <xacro:property name="base_height" value="0.17" />
+  <xacro:property name="hip_mass" value="2.0" />
+  <xacro:property name="hip_length" value="0.13" />
+  <xacro:property name="hip_width" value="0.09" />
+  <xacro:property name="hip_height" value="0.09" />
+  <xacro:property name="upper_leg_mass" value="1.0" />
+  <xacro:property name="upper_leg_length" value="0.076" />
+  <xacro:property name="upper_leg_width" value="0.076" />
+  <xacro:property name="upper_leg_height" value="0.425" />
+  <xacro:property name="lower_leg_mass" value="0.5" />
+  <xacro:property name="lower_leg_length" value="0.035" />
+  <xacro:property name="lower_leg_width" value="0.045" />
+  <xacro:property name="lower_leg_height" value="0.42" />
   <xacro:macro name="spot_base">
     <link name="base_link"/>
@@ -15,10 +38,12 @@
         <collision>
             <geometry>
-                <mesh filename="package://hector_spot_description/meshes/body_collision.stl" />
+              <mesh filename="package://hector_spot_description/meshes/body_collision.stl" /> <!-- TODO replace with primitive -->
             </geometry>
         </collision>
         <inertial>
-             <mass value="16.25" />
-             <inertia  ixx="0.085" ixy="0.0"  ixz="0.0"  iyy="1.045"  iyz="0.0"  izz="1.042" />
+            <mass value="${base_mass}"/>
+            <inertia ixx="${(1/12) * base_mass * (base_width * base_width + base_height * base_height)}" ixy="0.0" ixz="0.0"
+                        iyy="${(1/12) * base_mass * (base_length * base_length + base_height * base_height)}" iyz="0.0"
+                        izz="${(1/12) * base_mass * (base_length * base_length + base_width * base_width)}" />
         </inertial>
     </link>
@@ -35,280 +60,9 @@
         <child link="rear_rail" />
     </joint>
-    <link name="front_left_hip">
-        <visual>
-            <geometry>
-                <mesh filename="package://hector_spot_description/meshes/front_left_hip.dae" />
-            </geometry>
-        </visual>
-        <collision>
-            <geometry>
-                <mesh filename="package://hector_spot_description/meshes/front_left_hip_collision.stl" />
-            </geometry>
-        </collision>
-        <inertial>
-            <mass value="1.5" />
-            <inertia  ixx="0.0605" ixy="0.0"  ixz="0.0"  iyy="0.0"  iyz="0.0"  izz="0.0" />
-        </inertial>
-    </link>
-    <joint name="front_left_hip_x" type="revolute">
-        <origin xyz="0.29785 0.05500 0.00000" rpy="0 0 0" />
-        <axis xyz="1 0 0" />
-        <parent link="body" />
-        <child link="front_left_hip" />
-        <limit effort="1000" velocity="1000.00" lower="-0.78539816339744827899" upper="0.78539816339744827899" />
-    </joint>
-    <link name="front_left_upper_leg">
-        <visual>
-            <geometry>
-                <mesh filename="package://hector_spot_description/meshes/front_left_upper_leg.dae" />
-            </geometry>
-        </visual>
-        <collision>
-            <geometry>
-                <mesh filename="package://hector_spot_description/meshes/front_left_upper_leg_collision.stl" />
-            </geometry>
-        </collision>
-        <inertial>
-            <mass value="1.5" />
-            <inertia  ixx="0.0" ixy="0.0"  ixz="0.0"  iyy="0.05"  iyz="0.0"  izz="0.0" />
-        </inertial>
-    </link>
-    <joint name="front_left_hip_y" type="revolute">
-        <origin xyz="0.0 0.110945 0.0" rpy="0 0 0" />
-        <axis xyz="0 1 0" />
-        <parent link="front_left_hip" />
-        <child link="front_left_upper_leg" />
-        <limit effort="1000" velocity="1000.00" lower="-0.89884456477707963539" upper="2.2951079663725435509" />
-    </joint>
-    <link name="front_left_lower_leg">
-        <visual>
-            <geometry>
-                <mesh filename="package://hector_spot_description/meshes/front_left_lower_leg.dae" />
-            </geometry>
-        </visual>
-        <collision>
-            <geometry>
-                <mesh filename="package://hector_spot_description/meshes/front_left_lower_leg_collision.stl" />
-            </geometry>
-        </collision>
-        <inertial>
-          <mass value="1.0" />
-          <inertia  ixx="0.0" ixy="0.0"  ixz="0.0"  iyy="0.045"  iyz="0.0"  izz="0.0" />
-        </inertial>
-    </link>
-    <joint name="front_left_knee" type="revolute">
-        <origin xyz="0.025 0.000 -0.3205" rpy="0 0 0" />
-        <axis xyz="0 1 0" />
-        <parent link="front_left_upper_leg" />
-        <child link="front_left_lower_leg" />
-        <limit effort="1000" velocity="1000.00" lower="-2.7929" upper="-0.254801" />
-    </joint>
-    <link name="front_right_hip">
-        <visual>
-            <geometry>
-                <mesh filename="package://hector_spot_description/meshes/front_right_hip.dae" />
-            </geometry>
-        </visual>
-        <collision>
-            <geometry>
-                <mesh filename="package://hector_spot_description/meshes/front_right_hip_collision.stl" />
-            </geometry>
-        </collision>
-        <inertial>
-            <mass value="1.5" />
-            <inertia  ixx="0.0605" ixy="0.0"  ixz="0.0"  iyy="0.0"  iyz="0.0"  izz="0.0" />
-        </inertial>
-    </link>
-    <joint name="front_right_hip_x" type="revolute">
-        <origin xyz="0.29785 -0.05500 0.00000" rpy="0 0 0" />
-        <axis xyz="1 0 0" />
-        <parent link="body" />
-        <child link="front_right_hip" />
-        <limit effort="1000" velocity="1000.00" lower="-0.78539816339744827899" upper="0.78539816339744827899" />
-    </joint>
-    <link name="front_right_upper_leg">
-        <visual>
-            <geometry>
-                <mesh filename="package://hector_spot_description/meshes/front_right_upper_leg.dae" />
-            </geometry>
-        </visual>
-        <collision>
-            <geometry>
-                <mesh filename="package://hector_spot_description/meshes/front_right_upper_leg_collision.stl" />
-            </geometry>
-        </collision>
-        <inertial>
-            <mass value="1.5" />
-            <inertia  ixx="0.0" ixy="0.0"  ixz="0.0"  iyy="0.05"  iyz="0.0"  izz="0.0" />
-        </inertial>
-    </link>
-    <joint name="front_right_hip_y" type="revolute">
-        <origin xyz="0.0 -0.110945 0.0" rpy="0 0 0" />
-        <axis xyz="0 1 0" />
-        <parent link="front_right_hip" />
-        <child link="front_right_upper_leg" />
-        <limit effort="1000" velocity="1000.00" lower="-0.89884456477707963539" upper="2.2951079663725435509" />
-    </joint>
-    <link name="front_right_lower_leg">
-        <visual>
-            <geometry>
-                <mesh filename="package://hector_spot_description/meshes/front_right_lower_leg.dae" />
-            </geometry>
-        </visual>
-        <collision>
-            <geometry>
-                <mesh filename="package://hector_spot_description/meshes/front_right_lower_leg_collision.stl" />
-            </geometry>
-        </collision>
-        <inertial>
-            <mass value="1.0" />
-            <inertia  ixx="0.0" ixy="0.0"  ixz="0.0"  iyy="0.045"  iyz="0.0"  izz="0.0" />
-        </inertial>
-    </link>
-    <joint name="front_right_knee" type="revolute">
-        <origin xyz="0.025 0.000 -0.3205" rpy="0 0 0" />
-        <axis xyz="0 1 0" />
-        <parent link="front_right_upper_leg" />
-        <child link="front_right_lower_leg" />
-        <limit effort="1000" velocity="1000.00" lower="-2.7929" upper="-0.247563" />
-    </joint>
-    <link name="rear_left_hip">
-        <visual>
-            <geometry>
-                <mesh filename="package://hector_spot_description/meshes/rear_left_hip.dae" />
-            </geometry>
-        </visual>
-        <collision>
-            <geometry>
-                <mesh filename="package://hector_spot_description/meshes/rear_left_hip_collision.stl" />
-            </geometry>
-        </collision>
-        <inertial>
-            <mass value="1.5" />
-            <inertia  ixx="0.0605" ixy="0.0"  ixz="0.0"  iyy="0.0"  iyz="0.0"  izz="0.0" />
-        </inertial>
-    </link>
-    <joint name="rear_left_hip_x" type="revolute">
-        <origin xyz="-0.29785 0.05500 0.00000" rpy="0 0 0" />
-        <axis xyz="1 0 0" />
-        <parent link="body" />
-        <child link="rear_left_hip" />
-        <limit effort="1000" velocity="1000.00" lower="-0.78539816339744827899" upper="0.78539816339744827899" />
-    </joint>
-    <link name="rear_left_upper_leg">
-        <visual>
-            <geometry>
-                <mesh filename="package://hector_spot_description/meshes/rear_left_upper_leg.dae" />
-            </geometry>
-        </visual>
-        <collision>
-            <geometry>
-                <mesh filename="package://hector_spot_description/meshes/rear_left_upper_leg_collision.stl" />
-            </geometry>
-        </collision>
-        <inertial>
-            <mass value="1.5" />
-            <inertia  ixx="0.0" ixy="0.0"  ixz="0.0"  iyy="0.05"  iyz="0.0"  izz="0.0" />
-        </inertial>
-    </link>
-    <joint name="rear_left_hip_y" type="revolute">
-        <origin xyz="0.0 0.110945 0.0" rpy="0 0 0" />
-        <axis xyz="0 1 0" />
-        <parent link="rear_left_hip" />
-        <child link="rear_left_upper_leg" />
-        <limit effort="1000" velocity="1000.00" lower="-0.89884456477707963539" upper="2.2951079663725435509" />
-    </joint>
-    <link name="rear_left_lower_leg">
-        <visual>
-            <geometry>
-                <mesh filename="package://hector_spot_description/meshes/rear_left_lower_leg.dae" />
-            </geometry>
-        </visual>
-        <collision>
-            <geometry>
-                <mesh filename="package://hector_spot_description/meshes/rear_left_lower_leg_collision.stl" />
-            </geometry>
-        </collision>
-        <inertial>
-            <mass value="1.0" />
-            <inertia  ixx="0.0" ixy="0.0"  ixz="0.0"  iyy="0.045"  iyz="0.0"  izz="0.0" />
-        </inertial>
-    </link>
-    <joint name="rear_left_knee" type="revolute">
-        <origin xyz="0.025 0.000 -0.3205" rpy="0 0 0" />
-        <axis xyz="0 1 0" />
-        <parent link="rear_left_upper_leg" />
-        <child link="rear_left_lower_leg" />
-        <limit effort="1000" velocity="1000.00" lower="-2.7929" upper="-0.267153" />
-    </joint>
-    <link name="rear_right_hip">
-        <visual>
-            <geometry>
-                <mesh filename="package://hector_spot_description/meshes/rear_right_hip.dae" />
-            </geometry>
-        </visual>
-        <collision>
-            <geometry>
-                <mesh filename="package://hector_spot_description/meshes/rear_right_hip_collision.stl" />
-            </geometry>
-        </collision>
-        <inertial>
-            <mass value="1.5" />
-            <inertia  ixx="0.0605" ixy="0.0"  ixz="0.0"  iyy="0.0"  iyz="0.0"  izz="0.0" />
-        </inertial>
-    </link>
-    <joint name="rear_right_hip_x" type="revolute">
-        <origin xyz="-0.29785 -0.05500 0.00000" rpy="0 0 0" />
-        <axis xyz="1 0 0" />
-        <parent link="body" />
-        <child link="rear_right_hip" />
-        <limit effort="1000" velocity="1000.00" lower="-0.78539816339744827899" upper="0.78539816339744827899" />
-    </joint>
-    <link name="rear_right_upper_leg">
-        <visual>
-            <geometry>
-                <mesh filename="package://hector_spot_description/meshes/rear_right_upper_leg.dae" />
-            </geometry>
-        </visual>
-        <collision>
-            <geometry>
-                <mesh filename="package://hector_spot_description/meshes/rear_right_upper_leg_collision.stl" />
-            </geometry>
-        </collision>
-        <inertial>
-            <mass value="1.5" />
-            <inertia  ixx="0.0" ixy="0.0"  ixz="0.0"  iyy="0.05"  iyz="0.0"  izz="0.0" />
-        </inertial>
-    </link>
-    <joint name="rear_right_hip_y" type="revolute">
-        <origin xyz="0.0 -0.110945 0.0" rpy="0 0 0" />
-        <axis xyz="0 1 0" />
-        <parent link="rear_right_hip" />
-        <child link="rear_right_upper_leg" />
-        <limit effort="1000" velocity="1000.00" lower="-0.89884456477707963539" upper="2.2951079663725435509" />
-    </joint>
-    <link name="rear_right_lower_leg">
-        <visual>
-            <geometry>
-                <mesh filename="package://hector_spot_description/meshes/rear_right_lower_leg.dae" />
-            </geometry>
-        </visual>
-        <collision>
-            <geometry>
-                <mesh filename="package://hector_spot_description/meshes/rear_right_lower_leg_collision.stl" />
-            </geometry>
-        </collision>
-        <inertial>
-            <mass value="1.0" />
-            <inertia  ixx="0.0" ixy="0.0"  ixz="0.0"  iyy="0.045"  iyz="0.0"  izz="0.0" />
-        </inertial>
-    </link>
-    <joint name="rear_right_knee" type="revolute">
-        <origin xyz="0.025 0.000 -0.3205" rpy="0 0 0" />
-        <axis xyz="0 1 0" />
-        <parent link="rear_right_upper_leg" />
-        <child link="rear_right_lower_leg" />
-        <limit effort="1000" velocity="1000.00" lower="-2.7929" upper="-0.257725" />
-    </joint>
+    <!-- Legs -->
+    <xacro:spot_leg leg_name="front_left"/>
+    <xacro:spot_leg leg_name="front_right"/>
+    <xacro:spot_leg leg_name="rear_left"/>
+    <xacro:spot_leg leg_name="rear_right"/>
   </xacro:macro>
 </robot>

Commit message: Refactored left/right leg parameters

File: hector_spot_description/urdf/spot_base.urdf.xacro (robot description, xacro)
@@ -65,4 +65,8 @@
     <xacro:spot_leg leg_name="rear_left"/>
     <xacro:spot_leg leg_name="rear_right"/>
+    <xacro:spot_leg leg_name="front_left" front="1" left="1"/>
+    <xacro:spot_leg leg_name="front_right" front="1" left="-1"/>
+    <xacro:spot_leg leg_name="rear_left" front="-1" left="1"/>
+    <xacro:spot_leg leg_name="rear_right" front="-1" left="-1"/>
   </xacro:macro>
 </robot>

File: hector_spot_description/urdf/spot_leg.urdf.xacro (robot description, xacro)
@@ -3,20 +3,6 @@
     <xacro:include filename="$(find hector_xacro_tools)/urdf/joint_macros.urdf.xacro" />
     <xacro:macro name="spot_leg" params="leg_name" >
-        <xacro:if value="${leg_name == 'front_left'}">
-            <xacro:property name="base_to_hip_xyz"            value="${base_to_hip_x} ${base_to_hip_y} 0" />
-            <xacro:property name="hip_to_upper_leg_xyz"       value="0 ${hip_to_upper_leg_y} 0" />
-        </xacro:if>
-        <xacro:if value="${leg_name == 'front_right'}">
-            <xacro:property name="base_to_hip_xyz"            value="${base_to_hip_x} -${base_to_hip_y} 0" />
-            <xacro:property name="hip_to_upper_leg_xyz"       value="0 -${hip_to_upper_leg_y} 0" />
-        </xacro:if>
-        <xacro:if value="${leg_name == 'rear_left'}">
-            <xacro:property name="base_to_hip_xyz"            value="-${base_to_hip_x} ${base_to_hip_y} 0" />
-            <xacro:property name="hip_to_upper_leg_xyz"       value="0 ${hip_to_upper_leg_y} 0" />
-        </xacro:if>
-        <xacro:if value="${leg_name == 'rear_right'}">
-            <xacro:property name="base_to_hip_xyz"            value="-${base_to_hip_x} -${base_to_hip_y} 0" />
-            <xacro:property name="hip_to_upper_leg_xyz"       value="0 -${hip_to_upper_leg_y} 0" />
-        </xacro:if>
+        <xacro:property name="base_to_hip_xyz"            value="${front * base_to_hip_x} ${left * base_to_hip_y} 0" />
+        <xacro:property name="hip_to_upper_leg_xyz"       value="0 ${left * hip_to_upper_leg_y} 0" />
         <link name="${leg_name}_hip">
             <visual>

Commit message: Moved parameters to legs file

File: hector_spot_description/urdf/spot_base.urdf.xacro (robot description, xacro)
@@ -12,16 +12,4 @@
   <xacro:property name="base_width" value="0.21" />
   <xacro:property name="base_height" value="0.17" />
-  <xacro:property name="hip_mass" value="2.0" />
-  <xacro:property name="hip_length" value="0.13" />
-  <xacro:property name="hip_width" value="0.09" />
-  <xacro:property name="hip_height" value="0.09" />
-  <xacro:property name="upper_leg_mass" value="1.0" />
-  <xacro:property name="upper_leg_length" value="0.076" />
-  <xacro:property name="upper_leg_width" value="0.076" />
-  <xacro:property name="upper_leg_height" value="0.425" />
-  <xacro:property name="lower_leg_mass" value="0.5" />
-  <xacro:property name="lower_leg_length" value="0.035" />
-  <xacro:property name="lower_leg_width" value="0.045" />
-  <xacro:property name="lower_leg_height" value="0.42" />
   <xacro:macro name="spot_base">
     <link name="base_link"/>

File: hector_spot_description/urdf/spot_leg.urdf.xacro (robot description, xacro)
@@ -2,4 +2,16 @@
 <robot xmlns:xacro="http://ros.org/wiki/xacro">
     <xacro:include filename="$(find hector_xacro_tools)/urdf/joint_macros.urdf.xacro" />
+    <xacro:property name="hip_mass" value="2.0" />
+    <xacro:property name="hip_length" value="0.13" />
+    <xacro:property name="hip_width" value="0.09" />
+    <xacro:property name="hip_height" value="0.09" />
+    <xacro:property name="upper_leg_mass" value="1.0" />
+    <xacro:property name="upper_leg_length" value="0.076" />
+    <xacro:property name="upper_leg_width" value="0.076" />
+    <xacro:property name="upper_leg_height" value="0.425" />
+    <xacro:property name="lower_leg_mass" value="0.5" />
+    <xacro:property name="lower_leg_length" value="0.035" />
+    <xacro:property name="lower_leg_width" value="0.045" />
+    <xacro:property name="lower_leg_height" value="0.42" />
     <xacro:macro name="spot_leg" params="leg_name front left" >
         <xacro:property name="base_to_hip_xyz"            value="${front * base_to_hip_x} ${left * base_to_hip_y} 0" />
