Commit message: Added collision geometry with primitives

File: hector_spot_description/urdf/spot_base.urdf.xacro (robot description, xacro)
@@ -26,5 +26,6 @@
         <collision>
             <geometry>
-              <mesh filename="package://hector_spot_description/meshes/body_collision.stl" /> <!-- TODO replace with primitive -->
+<!--               <mesh filename="package://hector_spot_description/meshes/body_collision.stl" />  -->
+                <box size="0.872 0.239 0.195" />
             </geometry>
         </collision>

File: hector_spot_description/urdf/spot_leg.urdf.xacro (robot description, xacro)
@@ -3,7 +3,7 @@
     <xacro:include filename="$(find hector_xacro_tools)/urdf/joint_macros.urdf.xacro" />
     <xacro:property name="hip_mass" value="2.0" />
-    <xacro:property name="hip_length" value="0.13" />
-    <xacro:property name="hip_width" value="0.09" />
-    <xacro:property name="hip_height" value="0.09" />
+    <xacro:property name="hip_length" value="0.142" />
+    <xacro:property name="hip_width" value="0.1" />
+    <xacro:property name="hip_height" value="0.0941" />
     <xacro:property name="upper_leg_mass" value="1.0" />
     <xacro:property name="upper_leg_length" value="0.076" />
@@ -24,9 +24,12 @@
             </visual>
             <collision>
+                <origin xyz="${front * -0.023792} ${left * 0.011698} 0.000026 " rpy="0 0 0" />
                 <geometry>
-                    <mesh filename="package://hector_spot_description/meshes/${leg_name}_hip_collision.stl" /> <!-- TODO replace with primitive -->
+<!--                     <mesh filename="package://hector_spot_description/meshes/${leg_name}_hip_collision.stl" />  -->
+                  <box size="${hip_length} ${hip_width} ${hip_height}" />
                 </geometry>
             </collision>
             <inertial>
+                <origin xyz="${front * -0.023792} ${left * 0.011698} 0.000026 " rpy="0 0 0" />
                 <mass value="${hip_mass}"/>
                 <inertia ixx="${(1/12) * hip_mass * (hip_width * hip_width + hip_height * hip_height)}" ixy="0.0" ixz="0.0"
@@ -49,6 +52,8 @@
             </visual>
             <collision>
+                <origin xyz="0 0 -0.14" rpy="0 0 0" />
                 <geometry>
-                    <mesh filename="package://hector_spot_description/meshes/${leg_name}_upper_leg_collision.stl" /> <!-- TODO replace with primitive -->
+<!--                     <mesh filename="package://hector_spot_description/meshes/${leg_name}_upper_leg_collision.stl" />  -->
+                    <box size="${upper_leg_length} ${upper_leg_width} ${upper_leg_height}" />
                 </geometry>
             </collision>

Commit message: collision tuning

File: hector_spot_description/urdf/spot_base.urdf.xacro (robot description, xacro)
@@ -9,5 +9,5 @@
   <xacro:property name="lower_leg_to_foot_z" value="0.37" />
   <xacro:property name="base_mass" value="16.0" />
-  <xacro:property name="base_length" value="0.86" />
+  <xacro:property name="base_length" value="0.872" />
   <xacro:property name="base_width" value="0.21" />
   <xacro:property name="base_height" value="0.17" />
@@ -25,10 +25,12 @@
         </visual>
         <collision>
+            <origin xyz="0.006 0 0" rpy="0 0 0" />
             <geometry>
 <!--               <mesh filename="package://hector_spot_description/meshes/body_collision.stl" />  -->
-                <box size="0.872 0.239 0.195" />
+                <box size="${base_length} ${base_width} ${base_height}" />
             </geometry>
         </collision>
         <inertial>
+            <origin xyz="0.006 0 0" rpy="0 0 0" />
             <mass value="${base_mass}"/>
             <inertia ixx="${(1/12) * base_mass * (base_width * base_width + base_height * base_height)}" ixy="0.0" ixz="0.0"
