Commit message: Added spot cam payload

File: hector_spot_description/urdf/spot_macro.urdf.xacro (robot description, xacro)
@@ -3,9 +3,13 @@
   <xacro:include filename="$(find hector_spot_description)/urdf/spot_base.urdf.xacro"/>
   <xacro:include filename="$(find hector_spot_description)/urdf/spot_lidar_payload.urdf.xacro"/>
-  <xacro:macro name="spot_macro" params="lidar_payload:=false">
+  <xacro:include filename="$(find hector_spot_description)/urdf/spot_cam_payload.urdf.xacro"/>
+  <xacro:macro name="spot_macro" params="lidar_payload:=false cam_payload:=false">
     <xacro:spot_base/>
     <xacro:if value="${lidar_payload}">
       <xacro:spot_lidar_payload/>
     </xacro:if>
+    <xacro:if value="${cam_payload}">
+      <xacro:spot_cam_payload/>
+    </xacro:if>
   </xacro:macro>
 </robot>
