Commit message: Fixed links

File: hector_spot_description/urdf/spot_leg.urdf.xacro (robot description, xacro)
@@ -21,10 +21,10 @@
             <visual>
                 <geometry>
-                    <mesh filename="package://spot_description/meshes/${leg_name}_hip.dae" />
+                    <mesh filename="package://hector_spot_description/meshes/${leg_name}_hip.dae" />
                 </geometry>
             </visual>
             <collision>
                 <geometry>
-                    <mesh filename="package://spot_description/meshes/${leg_name}_hip_collision.stl" /> <!-- TODO replace with primitive -->
+                    <mesh filename="package://hector_spot_description/meshes/${leg_name}_hip_collision.stl" /> <!-- TODO replace with primitive -->
                 </geometry>
             </collision>
@@ -46,10 +46,10 @@
             <visual>
                 <geometry>
-                    <mesh filename="package://spot_description/meshes/${leg_name}_upper_leg.dae" />
+                    <mesh filename="package://hector_spot_description/meshes/${leg_name}_upper_leg.dae" />
                 </geometry>
             </visual>
             <collision>
                 <geometry>
-                    <mesh filename="package://spot_description/meshes/${leg_name}_upper_leg_collision.stl" /> <!-- TODO replace with primitive -->
+                    <mesh filename="package://hector_spot_description/meshes/${leg_name}_upper_leg_collision.stl" /> <!-- TODO replace with primitive -->
                 </geometry>
             </collision>
@@ -72,10 +72,10 @@
             <visual>
                 <geometry>
-                    <mesh filename="package://spot_description/meshes/${leg_name}_lower_leg.dae" />
+                    <mesh filename="package://hector_spot_description/meshes/${leg_name}_lower_leg.dae" />
                 </geometry>
             </visual>
             <collision>
                 <geometry>
-                    <mesh filename="package://spot_description/meshes/${leg_name}_lower_leg_collision.stl" scale="0.82 0.97 0.98"/> <!-- TODO replace with primitive -->
+                    <mesh filename="package://hector_spot_description/meshes/${leg_name}_lower_leg_collision.stl" scale="0.82 0.97 0.98"/> <!-- TODO replace with primitive -->
                 </geometry>
             </collision>

Commit message: Replaced transmission with macro

File: hector_spot_description/urdf/spot_leg.urdf.xacro (robot description, xacro)
@@ -1,4 +1,5 @@
 <?xml version="1.0"?>
 <robot xmlns:xacro="http://ros.org/wiki/xacro">
+    <xacro:include filename="$(find hector_xacro_tools)/urdf/joint_macros.urdf.xacro" />
     <xacro:macro name="spot_leg" params="leg_name" >
         <xacro:if value="${leg_name == 'front_left'}">
@@ -109,34 +110,7 @@
             <origin xyz="0 0 -${lower_leg_to_foot_z}" rpy="0 0 0" />
         </joint>
-        <transmission name="${leg_name}_hip_x_trans">
-            <type>transmission_interface/SimpleTransmission</type>
-            <joint name="${leg_name}_hip_x">
-                <hardwareInterface>hardware_interface/EffortJointInterface</hardwareInterface>
-            </joint>
-            <actuator name="${leg_name}_hip_x_actuator">
-                <hardwareInterface>hardware_interface/EffortJointInterface</hardwareInterface>
-                <mechanicalReduction>1</mechanicalReduction>
-            </actuator>
-        </transmission>
-        <transmission name="${leg_name}_hip_y_trans">
-            <type>transmission_interface/SimpleTransmission</type>
-            <joint name="${leg_name}_hip_y">
-                <hardwareInterface>hardware_interface/EffortJointInterface</hardwareInterface>
-            </joint>
-            <actuator name="${leg_name}_hip_y_actuator">
-                <hardwareInterface>hardware_interface/EffortJointInterface</hardwareInterface>
-                <mechanicalReduction>1</mechanicalReduction>
-            </actuator>
-        </transmission>
-        <transmission name="${leg_name}_knee_trans">
-            <type>transmission_interface/SimpleTransmission</type>
-            <joint name="${leg_name}_knee">
-                <hardwareInterface>hardware_interface/EffortJointInterface</hardwareInterface>
-            </joint>
-            <actuator name="${leg_name}_knee_actuator">
-                <hardwareInterface>hardware_interface/EffortJointInterface</hardwareInterface>
-                <mechanicalReduction>1</mechanicalReduction>
-            </actuator>
-        </transmission>
+        <xacro:joint_standard_transmission name="${leg_name}_hip_x"/>
+        <xacro:joint_standard_transmission name="${leg_name}_hip_y"/>
+        <xacro:joint_standard_transmission name="${leg_name}_knee"/>
     </xacro:macro>
 </robot>

Commit message: Replaced leg collisions with spheres

File: hector_spot_description/urdf/spot_leg.urdf.xacro (robot description, xacro)
@@ -42,5 +42,5 @@
             <parent link="body" />
             <child link="${leg_name}_hip" />
-            <limit effort="100" velocity="1000.00" lower="-0.78539816339744827899" upper="0.78539816339744827899" />
+            <limit effort="80" velocity="15" lower="-0.78539816339744827899" upper="0.78539816339744827899" />
         </joint>
         <link name="${leg_name}_upper_leg">
@@ -68,5 +68,5 @@
             <parent link="${leg_name}_hip" />
             <child link="${leg_name}_upper_leg" />
-            <limit effort="100" velocity="1000.00" lower="-0.89884456477707963539" upper="2.2951079663725435509" />
+            <limit effort="80" velocity="15" lower="-0.89884456477707963539" upper="2.2951079663725435509" />
         </joint>
         <link name="${leg_name}_lower_leg">
@@ -77,6 +77,7 @@
             </visual>
             <collision>
+                <origin xyz="0 0 -${lower_leg_to_foot_z - 0.04 + 0.003}" />
                 <geometry>
-                    <mesh filename="package://hector_spot_description/meshes/${leg_name}_lower_leg_collision.stl" scale="0.82 0.97 0.98"/> <!-- TODO replace with primitive -->
+                    <sphere radius="0.04" />
                 </geometry>
             </collision>
@@ -90,10 +91,10 @@
         </link>
          <gazebo reference="${leg_name}_lower_leg">
-            <kp>100000.0</kp>
-            <kd>1.0</kd>
+            <kp>1e+07</kp>
+            <kd>100.0</kd>
             <mu1>0.8</mu1>
             <mu2>0.8</mu2>
-            <maxVel>0.0</maxVel>
-            <minDepth>0.001</minDepth>
+<!--            <maxVel>0.0</maxVel>
+            <minDepth>0.001</minDepth>-->
         </gazebo>
         <joint name="${leg_name}_knee" type="revolute">
@@ -102,5 +103,5 @@
             <parent link="${leg_name}_upper_leg" />
             <child link="${leg_name}_lower_leg" />
-            <limit effort="100" velocity="1000.00" lower="-2.7929" upper="-0.254801" />
+            <limit effort="80" velocity="15" lower="-2.7929" upper="-0.254801" />
         </joint>
         <link name="${leg_name}_ee" />

Commit message: missing! Refactored left/right leg parameters

File: hector_spot_description/urdf/spot_leg.urdf.xacro (robot description, xacro)
@@ -2,5 +2,5 @@
 <robot xmlns:xacro="http://ros.org/wiki/xacro">
     <xacro:include filename="$(find hector_xacro_tools)/urdf/joint_macros.urdf.xacro" />
-    <xacro:macro name="spot_leg" params="leg_name" >
+    <xacro:macro name="spot_leg" params="leg_name front left" >
         <xacro:property name="base_to_hip_xyz"            value="${front * base_to_hip_x} ${left * base_to_hip_y} 0" />
         <xacro:property name="hip_to_upper_leg_xyz"       value="0 ${left * hip_to_upper_leg_y} 0" />

Commit message: Added collisions for handles on leg

File: hector_spot_description/urdf/spot_leg.urdf.xacro (robot description, xacro)
@@ -56,4 +56,11 @@
 <!--                     <mesh filename="package://hector_spot_description/meshes/${leg_name}_upper_leg_collision.stl" />  -->
                     <box size="${upper_leg_length} ${upper_leg_width} ${upper_leg_height}" />
+                </geometry>
+            </collision>
+            <!-- collision for handle -->
+              <collision>
+                <origin xyz="${-upper_leg_length/2 - 0.025} 0 0" rpy="0 0 0" />
+                <geometry>
+                    <box size="0.05 0.03 0.11" />
                 </geometry>
             </collision>
